Commit message: add launch file and fix inertia values for fingers

File: src/ur10e_gripper_description/urdf/simple_gripper.xacro (robot description, xacro)
@@ -8,5 +8,5 @@
       <visual>   <geometry><box size="0.06 0.08 0.03"/></geometry> <material name="grip_dark"/> </visual>
       <collision><geometry><box size="0.06 0.08 0.03"/></geometry> </collision>
-      <inertial> <mass value="1e-4"/> <inertia ixx="…" ixy="0" ixz="0" iyy="…" iyz="0" izz="…"/> </inertial>
+      <inertial> <mass value="1e-4"/> <inertia ixx="1e-4" ixy="0" ixz="0" iyy="1e-4" iyz="0" izz="1e-4"/> </inertial>
     </link>
     <joint name="gripper_base_joint" type="fixed">
@@ -17,5 +17,5 @@
       <visual>   <geometry><box size="0.012 0.012 0.05"/></geometry> <material name="grip_dark"/> </visual>
       <collision><geometry><box size="0.012 0.012 0.05"/></geometry> </collision>
-      <inertial> <mass value="0.05"/> <inertia ixx="1e-5" ixy="0" ixz="0" iyy="…" iyz="0" izz="…"/> </inertial>
+      <inertial> <mass value="0.05"/> <inertia ixx="1e-5" ixy="0" ixz="0" iyy="1e-5" iyz="0" izz="1e-5"/> </inertial>
     </link>
     <joint name="gripper_left_finger_joint" type="prismatic">
@@ -28,5 +28,5 @@
       <visual>   <geometry><box size="0.012 0.012 0.05"/></geometry> <material name="grip_dark"/> </visual>
       <collision><geometry><box size="0.012 0.012 0.05"/></geometry> </collision>
-      <inertial> <mass value="0.05"/> <inertia ixx="1e-5" ixy="0" ixz="0" iyy="…" iyz="0" izz="…"/> </inertial>
+      <inertial> <mass value="0.05"/> <inertia ixx="1e-5" ixy="0" ixz="0" iyy="1e-5" iyz="0" izz="1e-5"/> </inertial>
     </link>
     <joint name="gripper_right_finger_joint" type="prismatic">
