Commit message: feat: add robotiq 2f85 into the packages

File: src/ur10e_gripper_description/urdf/ur10e_ros2_control.xacro (robot description, xacro)
@@ -35,13 +35,35 @@
       <state_interface name="velocity"/>
     </joint>
-    <joint name="gripper_left_finger_joint">
+    <joint name="robotiq_85_left_knuckle_joint">
       <command_interface name="position"/>
-      <state_interface name="position"><param name="initial_value">0.0</param></state_interface>
+      <state_interface name="position"/>
       <state_interface name="velocity"/>
     </joint>
-    <joint name="gripper_right_finger_joint">
+    <joint name="robotiq_85_right_knuckle_joint">
+      <param name="mimic">robotiq_85_left_knuckle_joint</param>
+      <param name="multiplier">-1</param>
       <command_interface name="position"/>
-      <state_interface name="position"><param name="initial_value">0.0</param></state_interface>
+      <state_interface name="position"/>
       <state_interface name="velocity"/>
+    </joint>
+    <joint name="robotiq_85_left_inner_knuckle_joint">
+      <param name="mimic">robotiq_85_left_knuckle_joint</param>
+      <param name="multiplier">1</param>
+      <command_interface name="position"/><state_interface name="position"/><state_interface name="velocity"/>
+    </joint>
+    <joint name="robotiq_85_right_inner_knuckle_joint">
+      <param name="mimic">robotiq_85_left_knuckle_joint</param>
+      <param name="multiplier">-1</param>
+      <command_interface name="position"/><state_interface name="position"/><state_interface name="velocity"/>
+    </joint>
+    <joint name="robotiq_85_left_finger_tip_joint">
+      <param name="mimic">robotiq_85_left_knuckle_joint</param>
+      <param name="multiplier">-1</param>
+      <command_interface name="position"/><state_interface name="position"/><state_interface name="velocity"/>
+    </joint>
+    <joint name="robotiq_85_right_finger_tip_joint">
+      <param name="mimic">robotiq_85_left_knuckle_joint</param>
+      <param name="multiplier">1</param>
+      <command_interface name="position"/><state_interface name="position"/><state_interface name="velocity"/>
     </joint>
   </ros2_control>

File: src/ur10e_gripper_description/urdf/ur10e_with_gripper.urdf.xacro (robot description, xacro)
@@ -17,6 +17,12 @@
     <origin xyz="0 0 0" rpy="0 0 0"/>
   </xacro:ur_robot>
-  <xacro:include filename="simple_gripper.xacro"/>
-  <xacro:simple_gripper parent="tool0"/>
+  <!-- <xacro:include filename="simple_gripper.xacro"/>
+  <xacro:simple_gripper parent="tool0"/> -->
+  <xacro:include filename="$(find robotiq_description)/urdf/robotiq_2f_85_macro.urdf.xacro"/>
+  <xacro:robotiq_gripper
+    name="RobotiqGripper" prefix="" parent="tool0"
+    include_ros2_control="false">
+    <origin xyz="0 0 0" rpy="0 0 0"/>
+  </xacro:robotiq_gripper>
   <xacro:include filename="ur10e_ros2_control.xacro"/>
 </robot>
